Commit message: add color property to each link

File: urdf/robot.gazebo.xacro (robot description, xacro)
@@ -7,4 +7,5 @@
     <kd value="1.0"/>
     <fdir1 value="1 0 0"/>
+		<material>Gazebo/White</material>
     <turnGravityOff>false</turnGravityOff>
   </gazebo>
@@ -15,4 +16,5 @@
     <kd value="1.0"/>
     <fdir1 value="1 0 0"/>
+		<material>Gazebo/White</material>
     <turnGravityOff>false</turnGravityOff>
   </gazebo>
@@ -23,4 +25,5 @@
     <kd value="1.0"/>
     <fdir1 value="1 0 0"/>
+		<material>Gazebo/Red</material>
     <turnGravityOff>false</turnGravityOff>
   </gazebo>
